Commit message: capsense_update

File: assistive_gym/assistive_gym/envs/assets/stretch/stretch_uncalibrated_new.urdf (robot description, URDF)
Before this commit: robot stretch_description, 40 links, 39 joints
Links:
- added link camera_accel_frame
- added link camera_accel_optical_frame
- added link camera_gyro_frame
- added link camera_gyro_optical_frame
- added link caster_link, mass 0.01; collision sphere radius=0.032; visual mesh filename=meshes/omni_wheel_m.STL
- added link link_gripper_finger_left, mass 0.0476207785199474; collision mesh filename=meshes/link_gripper_finger_left.STL scale=0.9 1.0 1.0; visual mesh filename=meshes/link_gripper_finger_left.STL scale=0.9 1.0 1.0
- added link link_gripper_finger_right, mass 0.0476207785199481; collision mesh filename=meshes/link_gripper_finger_right.STL scale=0.9 1.0 1.0; visual mesh filename=meshes/link_gripper_finger_right.STL scale=0.9 1.0 1.0
- added link link_gripper_fingertip_left, mass 0.00382159917455729; collision mesh filename=meshes/link_gripper_fingertip_left.STL; visual mesh filename=meshes/link_gripper_fingertip_left.STL
- added link link_gripper_fingertip_right, mass 0.00382160037319545; collision mesh filename=meshes/link_gripper_fingertip_right.STL; visual mesh filename=meshes/link_gripper_fingertip_right.STL
- link camera_bottom_screw_frame: mass 0 -> None
- link camera_color_frame: mass 0 -> None
- link camera_color_optical_frame: mass 0 -> None
- link camera_depth_frame: mass 0 -> None
- link camera_depth_optical_frame: mass 0 -> None
- link camera_infra1_frame: mass 0 -> None
- link camera_infra1_optical_frame: mass 0 -> None
- link camera_infra2_frame: mass 0 -> None
- link camera_infra2_optical_frame: mass 0 -> None
- link camera_link: mass 0.564 -> 0.072; geometry collision box size=0.02505 0.09 0.025; visual mesh filename=package://realsense2_description/meshes/d435.dae
- link electrode1: geometry collision sphere radius=0.01; visual sphere radius=0.01
- link electrode2: geometry collision sphere radius=0.01; visual sphere radius=0.01
- link electrode3: geometry collision sphere radius=0.01; visual sphere radius=0.01
- link electrode4: geometry collision sphere radius=0.01; visual sphere radius=0.01
- link electrode5: geometry collision sphere radius=0.01; visual sphere radius=0.01
- link electrode6: geometry collision sphere radius=0.01; visual sphere radius=0.01
- link link_aruco_inner_wrist: mass 0.000225 -> 0
- link link_aruco_shoulder: mass 0.000399141592653546 -> 0
- link link_aruco_top_wrist: mass 0.000224999999999975 -> 0
- link link_grasp_center: mass 0.1 -> None
- link link_left_wheel: mass 0.00356714564938459 -> 0.01
- link link_right_wheel: mass 0.00356714564938475 -> 0.01
- link root_tool: mass 0.01 -> 0.1; geometry collision mesh filename=meshes/Tool1.STL scale=0.01 0.01 0.01; visual mesh filename=meshes/Tool1.STL scale=0.01 0.01 0.01
Joints:
- added joint camera_accel_joint: type fixed, parent camera_link, child camera_accel_frame, origin xyz=-0.01174 -0.00552 0.0051 rpy=0 0 0
- added joint camera_accel_optical_joint: type fixed, parent camera_accel_frame, child camera_accel_optical_frame, origin xyz=0 0 0 rpy=-1.57079632679 0 -1.57079632679
- added joint camera_gyro_joint: type fixed, parent camera_link, child camera_gyro_frame, origin xyz=-0.01174 -0.00552 0.0051 rpy=0 0 0
- added joint camera_gyro_optical_joint: type fixed, parent camera_gyro_frame, child camera_gyro_optical_frame, origin xyz=0 0 0 rpy=-1.57079632679 0 -1.57079632679
- added joint caster_joint: type fixed, parent base_link, child caster_link, origin xyz=-0.245 0.0 0.032 rpy=-1.57079632679 0 0, axis 0 0 1
- added joint joint_gripper_finger_left: type revolute, parent link_gripper, child link_gripper_finger_left, origin xyz=-0.047231 -0.010151 -0.04679 rpy=2.1762E-15 0.5236 3.1416, axis 0 0 1, limit lower=-0.6 upper=0.6 effort=100 velocity=1.0
- added joint joint_gripper_finger_right: type revolute, parent link_gripper, child link_gripper_finger_right, origin xyz=-0.047231 0.010049 -0.04679 rpy=3.1416 -0.5236 1.2943E-15, axis 0 0 1, limit lower=-0.6 upper=0.6 effort=100 velocity=1.0
- added joint joint_gripper_fingertip_left: type fixed, parent link_gripper_finger_left, child link_gripper_fingertip_left, origin xyz=0.171099 0.014912 0 rpy=-1.5708 -4.774E-15 -2.5545, axis 0 0 0
- added joint joint_gripper_fingertip_right: type fixed, parent link_gripper_finger_right, child link_gripper_fingertip_right, origin xyz=-0.171099 -0.014912 0 rpy=-1.5708 -2.0539E-15 0.58705, axis 0 0 0
- joint center_to_tool: axis (none) -> 0.0 0.0 0.0; origin xyz=0 0 0 rpy=0 0 0 -> xyz=-0.05 0.055 0.15 rpy=1.57079632679 2.09439510239 0; parent link_grasp_center -> link_gripper_fingertip_left
- joint joint_left_wheel: origin xyz=-0.003 0.15765 0.0508 rpy=-1.5707963267949 3.16227047920818E-31 7.88745438253713E-16 -> xyz=-0.00300000000001899 0.15765 0.0507999999999994 rpy=-1.5707963267949 3.16227047920818E-31 7.88745438253713E-16
- joint joint_right_wheel: origin xyz=-0.003 -0.15765 0.0508 rpy=-1.57079632679489 -1.11022302462516E-16 7.28583859910277E-17 -> xyz=-0.00300000000000034 -0.15765 0.0508000000000004 rpy=-1.57079632679489 -1.11022302462516E-16 7.28583859910277E-17
- joint root_to_electrode1: axis (none) -> 0.0 0.0 1.0; limit (none) -> lower=0.0 upper=1.1 effort=100.0 velocity=1.0; origin xyz=0.035, -0.05, -0.05 rpy=0 0 0 -> xyz=0.015 0.075 0 rpy=0 0 0; type fixed -> prismatic
- joint root_to_electrode2: axis (none) -> 0.0 0.0 1.0; limit (none) -> lower=0.0 upper=1.1 effort=100.0 velocity=1.0; origin xyz=-0.035 -0.05 -0.05 rpy=0 0 0 -> xyz=0.015 0.145 0 rpy=0 0 0; type fixed -> prismatic
- joint root_to_electrode3: axis (none) -> 0.0 0.0 1.0; limit (none) -> lower=0.0 upper=1.1 effort=100.0 velocity=1.0; origin xyz=0.035, 0, -0.05 rpy=0 0 0 -> xyz=0.070 0.075 0 rpy=0 0 0; type fixed -> prismatic
- joint root_to_electrode4: axis (none) -> 0.0 0.0 1.0; limit (none) -> lower=0.0 upper=1.1 effort=100.0 velocity=1.0; origin xyz=-0.035, 0, -0.05 rpy=0 0 0 -> xyz=0.070 0.145 0 rpy=0 0 0; type fixed -> prismatic
- joint root_to_electrode5: axis (none) -> 0.0 0.0 1.0; limit (none) -> lower=0.0 upper=1.1 effort=100.0 velocity=1.0; origin xyz=0.035, 0.05, -0.05 rpy=0 0 0 -> xyz=0.125 0.075 0 rpy=0 0 0; type fixed -> prismatic
- joint root_to_electrode6: axis (none) -> 0.0 0.0 1.0; limit (none) -> lower=0.0 upper=1.1 effort=100.0 velocity=1.0; origin xyz=-0.035, 0.05, -0.05 rpy=0 0 0 -> xyz=0.125 0.145 0 rpy=0 0 0; type fixed -> prismatic
